Commit message: Add MoveIt, aligned Nav2 map, status lights, auto doors, cameras & combined launches
New packages
- goliath_moveit_config: MoveIt 2 config for the 6-DOF arm (SRDF planning group
  arm_base_link->tool0, KDL IK, OMPL/RRTConnect, joint limits, controller bridge
  to arm_controller/follow_joint_trajectory, move_group + RViz launch incl.
  world->odom static TF so RViz has a valid fixed frame).
- goliath_lights: status-light node (levers latch by angle, buttons by rising
  edge) spawning colored markers on the switch wall.
- goliath_doors: auto sliding doors (proximity open/close via get/set_entity_state).

Description / world
- switch_wall model.sdf: joint_state_publisher plugin for the levers/buttons.
- datacenter.world: gazebo_ros_state plugin for the door node.
- goliath.urdf.xacro / goliath.gazebo.xacro: optional gripper + base cameras
  gated behind enable_cameras arg (default off).

Nav2 / mapping
- goliath_mapping/maps/datacenter: coordinate-aligned occupancy map generated
  from datacenter.world geometry (map frame == Gazebo world frame).
- nav2_params.yaml: odom topic -> /amr_controller/odom, robot_radius 0.30,
  AMCL set_initial_pose at the spawn pose (1,1).

Bringup
- switch_world_lights.launch.py: sim + lights + doors + teleop relay.
- switch_world_lights_cameras.launch.py: same, with cameras enabled.
- switch_world.launch.py / package.xml: enable_cameras passthrough + deps.

File: goliath_description/urdf/goliath.gazebo.xacro (robot description, xacro)
@@ -92,3 +92,41 @@
     </sensor>
   </gazebo>
+  <!-- Cameras (gated by enable_cameras). Standalone Gazebo sensors, independent
+       of ros2_control. Kept light (low res/rate) so rendering stays cheap. -->
+  <xacro:if value="$(arg enable_cameras)">
+    <!-- Gripper camera  ->  /arm_camera/image_raw -->
+    <gazebo reference="arm_camera_link">
+      <sensor type="camera" name="arm_camera">
+        <update_rate>10.0</update_rate>
+        <always_on>true</always_on>
+        <visualize>false</visualize>
+        <camera name="arm_camera">
+          <horizontal_fov>1.0472</horizontal_fov>
+          <image><width>320</width><height>240</height><format>R8G8B8</format></image>
+          <clip><near>0.02</near><far>50.0</far></clip>
+        </camera>
+        <plugin name="arm_camera_controller" filename="libgazebo_ros_camera.so">
+          <camera_name>arm_camera</camera_name>
+          <frame_name>arm_camera_optical</frame_name>
+        </plugin>
+      </sensor>
+    </gazebo>
+    <!-- Base camera  ->  /base_camera/image_raw -->
+    <gazebo reference="base_camera_link">
+      <sensor type="camera" name="base_camera">
+        <update_rate>10.0</update_rate>
+        <always_on>true</always_on>
+        <visualize>false</visualize>
+        <camera name="base_camera">
+          <horizontal_fov>1.3962</horizontal_fov>
+          <image><width>320</width><height>240</height><format>R8G8B8</format></image>
+          <clip><near>0.05</near><far>100.0</far></clip>
+        </camera>
+        <plugin name="base_camera_controller" filename="libgazebo_ros_camera.so">
+          <camera_name>base_camera</camera_name>
+          <frame_name>base_camera_optical</frame_name>
+        </plugin>
+      </sensor>
+    </gazebo>
+  </xacro:if>
 </robot>

File: goliath_description/urdf/goliath.urdf.xacro (robot description, xacro)
@@ -3,4 +3,6 @@
     <!--==========================================================MACROS====================================================================-->
     <xacro:arg name="is_sim" default="true"/>
+    <!-- Cameras off by default; the camera launch turns them on. -->
+    <xacro:arg name="enable_cameras" default="false"/>
     <!-- <xacro:property name="pi" value="3.14159265359" /> -->
     <xacro:include filename="$(find goliath_description)/urdf/goliath.gazebo.xacro" />
@@ -478,3 +480,50 @@
     <xacro:driving_wheel suffix="back_left" reflect="1" position="-0.19"/>
     <xacro:driving_wheel suffix="back_right" reflect="-1" position="-0.19"/>
+    <!--========================================================== CAMERAS ====================================================================-->
+    <!-- Two cameras (gripper + base). Gated by enable_cameras. These are only
+         camera links/sensors and do NOT touch the ros2_control block. -->
+    <xacro:if value="$(arg enable_cameras)">
+      <!-- Gripper camera (on tool0) -->
+      <link name="arm_camera_link">
+          <visual>
+              <origin xyz="0 0 0" rpy="0 0 0"/>
+              <geometry><box size="0.03 0.03 0.03"/></geometry>
+              <material name="black"/>
+          </visual>
+          <xacro:default_inertial mass="0.05"/>
+      </link>
+      <!-- Pushed 12 cm out along the tool axis so the camera clears the
+           gripper geometry (was buried inside it -> black image). -->
+      <joint name="arm_camera_joint" type="fixed">
+          <origin xyz="0 0 0.12" rpy="0 ${-pi/2} 0"/>
+          <parent link="tool0"/>
+          <child link="arm_camera_link"/>
+      </joint>
+      <link name="arm_camera_optical"/>
+      <joint name="arm_camera_optical_joint" type="fixed">
+          <origin xyz="0 0 0" rpy="${-pi/2} 0 ${-pi/2}"/>
+          <parent link="arm_camera_link"/>
+          <child link="arm_camera_optical"/>
+      </joint>
+      <!-- Base camera (front of base_link, looks forward +X) -->
+      <link name="base_camera_link">
+          <visual>
+              <origin xyz="0 0 0" rpy="0 0 0"/>
+              <geometry><box size="0.03 0.08 0.03"/></geometry>
+              <material name="black"/>
+          </visual>
+          <xacro:default_inertial mass="0.05"/>
+      </link>
+      <joint name="base_camera_joint" type="fixed">
+          <origin xyz="0.35 0 0.20" rpy="0 0 0"/>
+          <parent link="base_link"/>
+          <child link="base_camera_link"/>
+      </joint>
+      <link name="base_camera_optical"/>
+      <joint name="base_camera_optical_joint" type="fixed">
+          <origin xyz="0 0 0" rpy="${-pi/2} 0 ${-pi/2}"/>
+          <parent link="base_camera_link"/>
+          <child link="base_camera_optical"/>
+      </joint>
+    </xacro:if>
 </robot>
